Commit message: tested with images from camera mounted on ur5. need to decide if we want image generation of containing full robot pic or from mounted camera.

File: assets/walls/wall1.urdf (robot description, URDF)
Before this commit: robot simple_cuboid, 1 links, 0 joints
Links:
- link base_link: geometry collision box size=1.0 8.0 10.0; visual box size=1.0 8.0 10.0
